File: komagoma-2/komagoma-2.sch (EAGLE design)
At the start: 16 parts, among them IC1 TB6612FNGSSOP24, U1 XIAO-ESP32C3A

Commit message: order : .brd
Parts:
- added 5V, A0, D7: PINHD-1X1, Connector:PINHD-1X1
- added X1: JST-XH-02-PIN-LONG-PAD, Rembrandt Electronics - JST XH Connectors v1-0:JST-XH-02-PIN-LONG-PAD
- JP1: value JSTPH2 -> PINHD-1X4; device Tutorial - Fusion 360:JSTPH2 -> Connector:PINHD-1X4
Connections:
- new net 5V: 5V.1, U1.5V
- new net A0: A0.1, U1.GPIO2_A0_D0
- new net D7: D7.1, U1.GPIO20_D7_RX
- net +3V3: now also JP1.1
- net BAT-: now also X1-2.S; no longer JP1.1
- net BATT: now also X1-1.S; no longer JP1.2
- net GND: now also JP1.4
- net SCL: now also JP1.3
- net SDA: now also JP1.2
Other:
- note added: "JST"
Changed lines of the file:
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@@
 <class number="0" name="default" width="0.15" drill="0">
 </class>
-<class number="2" name="battery" width="0.6" drill="0">
+<class number="2" name="battery" width="0.5" drill="0">
 </class>
 <class number="3" name="VM" width="0.4" drill="0">
@@
 <part name="D1" library="LED" library_urn="urn:adsk.eagle:library:22900745" deviceset="WS2812B" device="" package3d_urn="urn:adsk.eagle:package:29365669/4"/>
 <part name="U$1" library="UTlibraries" deviceset="BNO055" device=""/>
-<part name="JP1" library="Tutorial - Fusion 360" library_urn="urn:adsk.eagle:library:16997205" deviceset="JSTPH2" device="" package3d_urn="urn:adsk.eagle:package:16863862/2"/>
 <part name="SUPPLY3" library="supply2" library_urn="urn:adsk.eagle:library:372" deviceset="GND" device=""/>
 <part name="SUPPLY4" library="supply2" library_urn="urn:adsk.eagle:library:372" deviceset="GND" device=""/>
@@
 <part name="SUPPLY11" library="supply2" library_urn="urn:adsk.eagle:library:372" deviceset="GND" device=""/>
 <part name="+3V5" library="supply1" library_urn="urn:adsk.eagle:library:371" deviceset="+3V3" device=""/>
+<part name="X1" library="Rembrandt Electronics - JST XH Connectors v1-0" deviceset="JST-XH-02-PIN" device="-LONG-PAD"/>
+<part name="JP1" library="Connector" library_urn="urn:adsk.eagle:library:16378166" deviceset="PINHD-1X4" device="" package3d_urn="urn:adsk.eagle:package:22407/2"/>
+<part name="SUPPLY12" library="supply2" library_urn="urn:adsk.eagle:library:372" deviceset="GND" device=""/>
+<part name="D7" library="Connector" library_urn="urn:adsk.eagle:library:16378166" deviceset="PINHD-1X1" device="" package3d_urn="urn:adsk.eagle:package:22485/2"/>
+<part name="5V" library="Connector" library_urn="urn:adsk.eagle:library:16378166" deviceset="PINHD-1X1" device="" package3d_urn="urn:adsk.eagle:package:22485/2"/>
+<part name="A0" library="Connector" library_urn="urn:adsk.eagle:library:16378166" deviceset="PINHD-1X1" device="" package3d_urn="urn:adsk.eagle:package:22485/2"/>
 </parts>
 <sheets>
@@
 <plain>
 <text x="-10.16" y="-43.18" size="2.54" layer="95">TB6612FNG</text>
+<text x="-66.04" y="-33.02" size="1.778" layer="95">JST</text>
 </plain>
 <instances>
@@
 </instance>
 <instance part="U$1" gate="G$1" x="-38.1" y="5.08" smashed="yes"/>
-<instance part="JP1" gate="G$1" x="-68.58" y="-30.48" smashed="yes" rot="MR180">
-<attribute name="VALUE" x="-72.39" y="-33.02" size="1.778" layer="96" rot="MR180"/>
-</instance>
 <instance part="SUPPLY3" gate="GND" x="25.4" y="-83.82" smashed="yes">
 <attribute name="VALUE" x="23.495" y="-86.995" size="1.778" layer="96"/>
@@
 <instance part="+3V5" gate="G$1" x="-71.12" y="-7.62" smashed="yes">
 <attribute name="VALUE" x="-68.58" y="-5.08" size="1.778" layer="96" rot="R180"/>
+</instance>
+<instance part="X1" gate="-2" x="-66.04" y="-30.48" smashed="yes">
+<attribute name="NAME" x="-63.5" y="-31.242" size="1.524" layer="95"/>
+</instance>
+<instance part="X1" gate="-1" x="-66.04" y="-27.94" smashed="yes">
+<attribute name="NAME" x="-63.5" y="-28.702" size="1.524" layer="95"/>
+</instance>
+<instance part="JP1" gate="A" x="-83.82" y="2.54" smashed="yes" rot="MR0">
+<attribute name="VALUE" x="-74.93" y="10.16" size="1.778" layer="96" rot="MR0"/>
+</instance>
+<instance part="SUPPLY12" gate="GND" x="-81.28" y="-5.08" smashed="yes"/>
+<instance part="D7" gate="G$1" x="-111.76" y="-48.26" smashed="yes" rot="R180">
+<attribute name="NAME" x="-105.41" y="-51.435" size="1.778" layer="95" rot="R180"/>
+<attribute name="VALUE" x="-105.41" y="-43.18" size="1.778" layer="96" rot="R180"/>
+</instance>
+<instance part="5V" gate="G$1" x="-106.68" y="-78.74" smashed="yes" rot="R270">
+<attribute name="NAME" x="-103.505" y="-72.39" size="1.778" layer="95" rot="R270"/>
+<attribute name="VALUE" x="-111.76" y="-72.39" size="1.778" layer="96" rot="R270"/>
+</instance>
+<instance part="A0" gate="G$1" x="-58.42" y="-78.74" smashed="yes" rot="R270">
+<attribute name="NAME" x="-55.245" y="-72.39" size="1.778" layer="95" rot="R270"/>
+<attribute name="VALUE" x="-63.5" y="-72.39" size="1.778" layer="96" rot="R270"/>
 </instance>
 </instances>
@@
 <pinref part="U$2" gate="G$1" pin="GND"/>
 <pinref part="SUPPLY11" gate="GND" pin="GND"/>
+</segment>
+<segment>
+<pinref part="JP1" gate="A" pin="4"/>
+<pinref part="SUPPLY12" gate="GND" pin="GND"/>
+<wire x1="-81.28" y1="0" x2="-81.28" y2="-2.54" width="0.1524" layer="91"/>
 </segment>
 </net>
@@
 <wire x1="-58.42" y1="-15.24" x2="-55.88" y2="-15.24" width="0.1524" layer="91"/>
 <junction x="-55.88" y="-15.24"/>
+<wire x1="-55.88" y1="0" x2="-73.66" y2="0" width="0.1524" layer="91"/>
+<wire x1="-73.66" y1="0" x2="-73.66" y2="2.54" width="0.1524" layer="91"/>
+<junction x="-55.88" y="0"/>
+<pinref part="JP1" gate="A" pin="3"/>
+<wire x1="-73.66" y1="2.54" x2="-81.28" y2="2.54" width="0.1524" layer="91"/>
 </segment>
 </net>
@@
 <wire x1="-58.42" y1="-12.7" x2="-53.34" y2="-12.7" width="0.1524" layer="91"/>
 <junction x="-53.34" y="-12.7"/>
+<pinref part="JP1" gate="A" pin="2"/>
+<wire x1="-81.28" y1="5.08" x2="-71.12" y2="5.08" width="0.1524" layer="91"/>
+<wire x1="-71.12" y1="5.08" x2="-71.12" y2="2.54" width="0.1524" layer="91"/>
+<wire x1="-71.12" y1="2.54" x2="-53.34" y2="2.54" width="0.1524" layer="91"/>
+<junction x="-53.34" y="2.54"/>
 </segment>
 </net>
 <net name="BAT-" class="2">
 <segment>
-<pinref part="JP1" gate="G$1" pin="1"/>
 <pinref part="U1" gate="G$1" pin="BATT-"/>
 <wire x1="-68.58" y1="-30.48" x2="-68.58" y2="-35.56" width="0.1524" layer="91"/>
 <wire x1="-68.58" y1="-35.56" x2="-69.85" y2="-35.56" width="0.1524" layer="91"/>
+<pinref part="X1" gate="-2" pin="S"/>
 </segment>
 </net>
 <net name="BATT" class="2">
 <segment>
-<pinref part="JP1" gate="G$1" pin="2"/>
 <pinref part="CONNECTOR1" gate="G$1" pin="1"/>
 <wire x1="-76.2" y1="-26.67" x2="-76.2" y2="-27.94" width="0.1524" layer="91"/>
 <wire x1="-76.2" y1="-27.94" x2="-68.58" y2="-27.94" width="0.1524" layer="91"/>
+<pinref part="X1" gate="-1" pin="S"/>
 </segment>
 </net>
@@
 <pinref part="U$1" gate="G$1" pin="VIN"/>
 <pinref part="+3V4" gate="G$1" pin="+3V3"/>
+<pinref part="JP1" gate="A" pin="1"/>
+<wire x1="-81.28" y1="7.62" x2="-50.8" y2="7.62" width="0.1524" layer="91"/>
+<junction x="-50.8" y="7.62"/>
 </segment>
 <segment>
@@
 </segment>
 </net>
+<net name="A0" class="0">
+<segment>
+<pinref part="U1" gate="G$1" pin="GPIO2_A0_D0"/>
+<pinref part="A0" gate="G$1" pin="1"/>
+<wire x1="-58.42" y1="-72.39" x2="-58.42" y2="-76.2" width="0.1524" layer="91"/>
+</segment>
+</net>
+<net name="5V" class="0">
+<segment>
+<pinref part="U1" gate="G$1" pin="5V"/>
+<pinref part="5V" gate="G$1" pin="1"/>
+<wire x1="-106.68" y1="-72.39" x2="-106.68" y2="-76.2" width="0.1524" layer="91"/>
+</segment>
+</net>
+<net name="D7" class="0">
+<segment>
+<pinref part="U1" gate="G$1" pin="GPIO20_D7_RX"/>
+<pinref part="D7" gate="G$1" pin="1"/>
+<wire x1="-106.68" y1="-49.53" x2="-109.22" y2="-49.53" width="0.1524" layer="91"/>
+<wire x1="-109.22" y1="-49.53" x2="-109.22" y2="-48.26" width="0.1524" layer="91"/>
+</segment>
+</net>
